Commit message: modifying urdf for gazebo ackerman plugin

File: src/segwayrmp_description/urdf/segwayrmp.urdf (robot description, URDF)
Before this commit: robot segwayrmp_description, 9 links, 8 joints
Links:
- removed link FrontPivot_Link
- removed link LeftFrontWheel_Link
- removed link LeftRearWheel_Link
- removed link RightFrontWheel_Link
- removed link RightRearWheel_Link
- removed link imu_link
- added link front_left_wheel_Link, mass 0.379124506048444; collision cylinder length=${wheel_length} radius=${wheel_radius}; visual cylinder length=${wheel_length} radius=${wheel_radius}
- added link front_pivot_Link, mass 0.636763996187421; collision cylinder length=0.44 radius=0.07; visual cylinder length=0.44 radius=0.07
- added link front_right_wheel_Link, mass 0.37912408551256; collision cylinder length=${wheel_length} radius=${wheel_radius}; visual cylinder length=${wheel_length} radius=${wheel_radius}
- added link rear_left_wheel_Link, mass 0.634779873374433; collision cylinder length=${wheel_length} radius=${wheel_radius}; visual cylinder length=${wheel_length} radius=${wheel_radius}
- added link rear_right_wheel_Link, mass 0.634778552429949; collision cylinder length=${wheel_length} radius=${wheel_radius}; visual cylinder length=${wheel_length} radius=${wheel_radius}
Joints:
- removed joint FrontPivot_joint
- removed joint LeftFrontWheel_joint
- removed joint LeftRearWheel_joint
- removed joint RightFrontWheel_joint
- removed joint RightRearWheel_joint
- removed joint imu_joint
- added joint front_left_wheel_joint: type continuous, parent front_pivot_Link, child front_left_wheel_Link, origin xyz=-0.092435 -0.06 0 rpy=2.9877 0 0, axis 1 0 0
- added joint front_pivot_joint: type revolute, parent base_link, child front_pivot_Link, origin xyz=0 0.46 0.15 rpy=1.5708 0 0, axis 0 -1 0, limit lower=-0.36 upper=0.36 effort=0 velocity=0
- added joint front_right_wheel_joint: type continuous, parent front_pivot_Link, child front_right_wheel_Link, origin xyz=0.099447 -0.06 0 rpy=-1.6671 0 3.1416, axis 1 0 0
- added joint rear_left_wheel_joint: type continuous, parent base_link, child rear_left_wheel_Link, origin xyz=-0.1 0.01 0.09 rpy=1.5708 0 0, axis 1 0 0
- added joint rear_right_wheel_joint: type continuous, parent base_link, child rear_right_wheel_Link, origin xyz=0.1 0.01 0.09 rpy=0.17453 0 -3.1416, axis 1 0 0

Commit message: Tuning for gazebo ackerman plugin

File: src/segwayrmp_description/urdf/segwayrmp.urdf (robot description, URDF)
Before this commit: robot segwayrmp_urdf, 8 links, 7 joints
Links:
- removed link world_link
- added link left_steering_link, mass 0.001
- added link steering_wheel_Link, mass 0.001
Joints:
- removed joint world_joint
- added joint left_steering_joint: type revolute, parent base_link, child left_steering_link, origin xyz=0 0.46 0.15 rpy=1.5708 0 0, axis 0 -1 0, limit lower=-0.36 upper=0.36 effort=0 velocity=0
- added joint steering_wheel_joint: type continuous, parent base_link, child steering_wheel_Link, origin xyz=0 0.46 0.15 rpy=1.5708 0 0, axis 0 -1 0
