Commit message: Set up the urdf and launch file for simulation

File: src/segwayrmp_description/urdf/segwayrmp.urdf.xacro (robot description, xacro)
@@ -1,53 +1,58 @@
 <?xml version="1.0" encoding="utf-8"?>
-<!-- This URDF was automatically created by SolidWorks to URDF Exporter! Originally created by Stephen Brawner (brawner@gmail.com)
+<!-- This URDF was automatically created by SolidWorks to URDF Exporter! Originally created by
+Stephen Brawner (brawner@gmail.com)
      Commit Version: 1.5.1-0-g916b5db  Build Version: 1.5.7152.31018
      For more information, please see http://wiki.ros.org/sw_urdf_exporter -->
-<robot
-  name="401pius">
-  <link
-    name="chejia_link">
-    <inertial>
-      <origin
-        xyz="0.00361762800581263 -0.133421165022722 0.0648164589836014"
+<robot name="segwayrmp_description" xmlns:xacro="http://ros.org/wiki/xacro">
+  <!-- Define robot constants -->
+  <xacro:property name="base_width" value="0.598" />
+  <xacro:property name="base_length" value="0.672" />
+  <xacro:property name="base_height" value="0.280" />
+  <!-- Dummy root link -->
+  <link name="world_link" />
+  <!-- Robot Base -->
+  <link name="base_link">
+    <inertial>
+      <origin
+        xyz="0 0.23 0.19"
         rpy="0 0 0" />
       <mass
         value="2.42397545608915" />
-      <inertia
-        ixx="0.0296962022350776"
-        ixy="2.4976120795965E-06"
-        ixz="-1.37689680267216E-05"
-        iyy="0.0331663553221158"
-        iyz="3.0593217918394E-05"
-        izz="0.00646533575042488" />
-    </inertial>
-    <visual>
-      <origin
-        xyz="0 0 0"
-        rpy="0 0 0" />
-      <geometry>
-        <mesh
-          filename="package://401pius/meshes/chejia_link.STL" />
-      </geometry>
-      <material
-        name="">
-        <color
-          rgba="0.792156862745098 0.819607843137255 0.933333333333333 1" />
-      </material>
-    </visual>
-    <collision>
-      <origin
-        xyz="0 0 0"
-        rpy="0 0 0" />
-      <geometry>
-        <mesh
-          filename="package://401pius/meshes/chejia_link.STL" />
-      </geometry>
-    </collision>
-  </link>
-  <link
-    name="zhuanxiangjia_Link">
-    <inertial>
-      <origin
-        xyz="0.00350625991709064 -0.184876810131571 -0.22368381667265"
+        <inertia ixx="0.0296962022350776" ixy="0" ixz="0"
+        iyy="0.00646533575042488" iyz="0" izz="0.0331663553221158" />
+    </inertial>
+    <visual>
+      <origin xyz="0 0.24 0.31" rpy="0 0 0" />
+      <geometry>
+        <mesh filename="package://segwayrmp_description/meshes/chejia_link.STL" />
+      </geometry>
+      <material name="">
+        <color rgba="0.792156862745098 0.819607843137255 0.933333333333333 1" />
+      </material>
+    </visual>
+    <collision>
+      <origin xyz="0 0.24 0.31" rpy="0 0 0" />
+      <geometry>
+        <mesh filename="package://segwayrmp_description/meshes/chejia_link.STL" />
+      </geometry>
+    </collision>
+  </link>
+  <!-- Fixed joint between world_link and base_link -->
+  <joint name="world_joint" type="fixed">
+    <parent link="world_link" />
+    <child link="base_link" />
+    <origin xyz="0 0 0" rpy="0 0 0" />
+  </joint>
+  <!-- Robot Footprint -->
+  <link name="base_footprint" />
+  <joint name="base_joint" type="fixed">
+    <parent link="base_link" />
+    <child link="base_footprint" />
+    <origin xyz="0.0 0.26 0" rpy="0 0 0" />
+  </joint>
+  <link name="FrontPivot_Link">
+    <inertial>
+      <origin
+        xyz="0.00350625991709064 0 0"
         rpy="0 0 0" />
       <mass
@@ -62,50 +67,36 @@
     </inertial>
     <visual>
-      <origin
-        xyz="0 0 0"
-        rpy="0 0 0" />
-      <geometry>
-        <mesh
-          filename="package://401pius/meshes/zhuanxiangjia_Link.STL" />
-      </geometry>
-      <material
-        name="">
-        <color
-          rgba="0.792156862745098 0.819607843137255 0.933333333333333 1" />
-      </material>
-    </visual>
-    <collision>
-      <origin
-        xyz="0 0 0"
-        rpy="0 0 0" />
-      <geometry>
-        <mesh
-          filename="package://401pius/meshes/zhuanxiangjia_Link.STL" />
-      </geometry>
-    </collision>
-  </link>
-  <joint
-    name="zhuanxiangjia_joint"
-    type="revolute">
-    <origin
-      xyz="0 0 0"
-      rpy="1.5708 0 0" />
-    <parent
-      link="chejia_link" />
-    <child
-      link="zhuanxiangjia_Link" />
-    <axis
-      xyz="0 -1 0" />
+      <origin xyz="0.0 0.16 0.22" rpy="0 0 0" />
+      <geometry>
+        <mesh
+          filename="package://segwayrmp_description/meshes/zhuanxiangjia_Link.STL" />
+      </geometry>
+      <material name="">
+        <color rgba="0.792156862745098 0.819607843137255 0.933333333333333 1" />
+      </material>
+    </visual>
+    <collision>
+      <origin xyz="0 0.16 0.22" rpy="0 0 0" />
+      <geometry>
+        <mesh filename="package://segwayrmp_description/meshes/zhuanxiangjia_Link.STL" />
+      </geometry>
+    </collision>
+  </link>
+  <joint name="FrontPivot_joint" type="revolute">
+    <origin xyz="0 0.46 0.15" rpy="1.5708 0 0" />
+    <parent link="base_link" />
+    <child link="FrontPivot_Link" />
+    <axis xyz="0 -1 0" />
     <limit
-      lower="0"
-      upper="0"
+      lower="-0.36"
+      upper="0.36"
       effort="0"
       velocity="0" />
   </joint>
   <link
-    name="zuoqianlun_Link">
-    <inertial>
-      <origin
-        xyz="-0.18003195018567 0.0161203758776952 -0.0161713179715041"
+    name="LeftFrontWheel_Link">
+    <inertial>
+      <origin
+        xyz="-0.21 0 0"
         rpy="0 0 0" />
       <mass
@@ -121,9 +112,9 @@
     <visual>
       <origin
-        xyz="0 0 0"
-        rpy="0 0 0" />
-      <geometry>
-        <mesh
-          filename="package://401pius/meshes/zuoqianlun_Link.STL" />
+        xyz="0.015 0 0"
+        rpy="0 0 0" />
+      <geometry>
+        <mesh
+          filename="package://segwayrmp_description/meshes/zuohoulun_Link.STL" />
       </geometry>
       <material
@@ -135,30 +126,30 @@
     <collision>
       <origin
-        xyz="0 0 0"
-        rpy="0 0 0" />
-      <geometry>
-        <mesh
-          filename="package://401pius/meshes/zuoqianlun_Link.STL" />
+        xyz="0.015 0 0"
+        rpy="0 0 0" />
+      <geometry>
+        <mesh
+          filename="package://segwayrmp_description/meshes/zuohoulun_Link.STL" />
       </geometry>
     </collision>
   </link>
   <joint
-    name="zuoqianlun_joint"
+    name="LeftFrontWheel_joint"
     type="continuous">
     <origin
-      xyz="-0.092435 -0.21283 -0.24243"
+      xyz="-0.092435 -0.06 -0.02"
       rpy="2.9877 0 0" />
     <parent
-      link="zhuanxiangjia_Link" />
+      link="FrontPivot_Link" />
     <child
-      link="zuoqianlun_Link" />
+      link="LeftFrontWheel_Link" />
     <axis
       xyz="1 0 0" />
   </joint>
   <link
-    name="youqianlun_Link">
-    <inertial>
-      <origin
-        xyz="-0.180031949902314 0.0161203458684245 -0.0161712883250444"
+    name="RightFrontWheel_Link">
+    <inertial>
+      <origin
+        xyz="-0.21 0.01 0"
         rpy="0 0 0" />
       <mass
@@ -174,9 +165,9 @@
     <visual>
       <origin
-        xyz="0 0 0"
-        rpy="0 0 0" />
-      <geometry>
-        <mesh
-          filename="package://401pius/meshes/youqianlun_Link.STL" />
+        xyz="0.015 0 0"
+        rpy="0 0 0" />
+      <geometry>
+        <mesh
+          filename="package://segwayrmp_description/meshes/zuohoulun_Link.STL" />
       </geometry>
       <material
@@ -188,27 +179,27 @@
     <collision>
       <origin
-        xyz="0 0 0"
-        rpy="0 0 0" />
-      <geometry>
-        <mesh
-          filename="package://401pius/meshes/youqianlun_Link.STL" />
+        xyz="0.015 0 0"
+        rpy="0 0 0" />
+      <geometry>
+        <mesh
+          filename="package://segwayrmp_description/meshes/zuohoulun_Link.STL" />
       </geometry>
     </collision>
   </link>
   <joint
-    name="youqianlun_joint"
+    name="RightFrontWheel_joint"
     type="continuous">
     <origin
-      xyz="0.099447 -0.24433 -0.20905"
+      xyz="0.099447 -0.06 0"
       rpy="-1.6671 0 3.1416" />
     <parent
-      link="zhuanxiangjia_Link" />
+      link="FrontPivot_Link" />
     <child
-      link="youqianlun_Link" />
+      link="RightFrontWheel_Link" />
     <axis
       xyz="1 0 0" />
   </joint>
   <link
-    name="zuohoulun_Link">
+    name="LeftRearWheel_Link">
     <inertial>
       <origin
@@ -227,9 +218,9 @@
     <visual>
       <origin
-        xyz="0 0 0"
-        rpy="0 0 0" />
-      <geometry>
-        <mesh
-          filename="package://401pius/meshes/zuohoulun_Link.STL" />
+        xyz="0.03 0 0"
+        rpy="0 0 0" />
+      <geometry>
+        <mesh
+          filename="package://segwayrmp_description/meshes/zuohoulun_Link.STL" />
       </geometry>
       <material
@@ -241,27 +232,27 @@
     <collision>
       <origin
-        xyz="0 0 0"
-        rpy="0 0 0" />
-      <geometry>
-        <mesh
-          filename="package://401pius/meshes/zuohoulun_Link.STL" />
+        xyz="0.03 0 0"
+        rpy="0 0 0" />
+      <geometry>
+        <mesh
+          filename="package://segwayrmp_description/meshes/zuohoulun_Link.STL" />
       </geometry>
     </collision>
   </link>
   <joint
-    name="zuohoulun_joint"
+    name="LeftRearWheel_joint"
     type="continuous">
     <origin
-      xyz="-0.058831 -0.23219 -0.22848"
+      xyz="-0.1 0.01 0.09"
       rpy="1.5708 0 0" />
     <parent
-      link="chejia_link" />
+      link="base_link" />
     <child
-      link="zuohoulun_Link" />
+      link="LeftRearWheel_Link" />
     <axis
       xyz="1 0 0" />
   </joint>
   <link
-    name="youhoulun_Link">
+    name="RightRearWheel_Link">
     <inertial>
       <origin
@@ -280,9 +271,9 @@
     <visual>
       <origin
-        xyz="0 0 0"
-        rpy="0 0 0" />
-      <geometry>
-        <mesh
-          filename="package://401pius/meshes/youhoulun_Link.STL" />
+        xyz="0.03 0 0"
+        rpy="0 0 0" />
+      <geometry>
+        <mesh
+          filename="package://segwayrmp_description/meshes/zuohoulun_Link.STL" />
       </geometry>
       <material
@@ -294,22 +285,22 @@
     <collision>
       <origin
-        xyz="0 0 0"
-        rpy="0 0 0" />
-      <geometry>
-        <mesh
-          filename="package://401pius/meshes/youhoulun_Link.STL" />
+        xyz="0.03 0 0"
+        rpy="0 0 0" />
+      <geometry>
+        <mesh
+          filename="package://segwayrmp_description/meshes/zuohoulun_Link.STL" />
       </geometry>
     </collision>
   </link>
   <joint
-    name="youhoulun_joint"
+    name="RightRearWheel_joint"
     type="continuous">
     <origin
-      xyz="0.065844 -0.23219 -0.22848"
+      xyz="0.1 0.01 0.09"
       rpy="0.17453 0 -3.1416" />
     <parent
-      link="chejia_link" />
+      link="base_link" />
     <child
-      link="youhoulun_Link" />
+      link="RightRearWheel_Link" />
     <axis
       xyz="1 0 0" />
