Commit message: Update urdf file path to use xacro extension and adjusted links and joints for steering using gazebo tricycle plugin

File: src/segwayrmp_description/urdf/segwayrmp.urdf.xacro (robot description, xacro)
@@ -4,12 +4,15 @@
      Commit Version: 1.5.1-0-g916b5db  Build Version: 1.5.7152.31018
      For more information, please see http://wiki.ros.org/sw_urdf_exporter -->
-<robot name="segwayrmp_description" xmlns:xacro="http://ros.org/wiki/xacro">
+<robot name="segwayrmp_urdf" xmlns:xacro="http://ros.org/wiki/xacro">
+  <xacro:arg name="robot_namespace" default="/" />
+  <xacro:include filename="$(find segwayrmp_description)/urdf/segwayrmp_xacro.xacro" />
+  <!-- <xacro:include filename="$(find segwayrmp_description)/urdf/segwayrmp_steering.xacro" /> -->
+  <xacro:include filename="$(find segwayrmp_description)/urdf/segwayrmp_ackerman.gazebo" />
   <!-- Define robot constants -->
   <xacro:property name="base_length" value="0.18" />
   <xacro:property name="base_width" value="0.61" />
   <xacro:property name="base_height" value="0.09" />
-  <xacro:arg name="robot_namespace" default="/" />
-  <!-- Dummy root link -->
-  <link name="world_link" />
+  <xacro:property name="wheel_length" value="0.05" />
+  <xacro:property name="wheel_radius" value="0.1" />
   <!-- Robot Base -->
   <link name="base_link">
@@ -25,6 +28,5 @@
       <origin xyz="0 0.24 0.21" rpy="0 0 0" />
       <geometry>
-        <!-- <mesh filename="package://segwayrmp_description/meshes/chejia_link.stl" /> -->
-        <box size="${base_length} ${base_width} ${base_height}"/>
+        <box size="${base_length} ${base_width} ${base_height}" />
       </geometry>
       <material name="">
@@ -35,71 +37,79 @@
       <origin xyz="0 0.24 0.21" rpy="0 0 0" />
       <geometry>
-        <!-- <mesh filename="package://segwayrmp_description/meshes/chejia_link.stl" /> -->
-        <box size="${base_length} ${base_width} ${base_height}"/>
-      </geometry>
-    </collision>
-  </link>
-  <!-- Fixed joint between world_link and base_link -->
-  <joint name="world_joint" type="fixed">
-    <parent link="world_link" />
-    <child link="base_link" />
-    <origin xyz="0 0 0" rpy="0 0 0" />
-  </joint>
-  <!-- Robot Footprint -->
-  <link name="base_footprint" />
-  <joint name="base_joint" type="fixed">
-    <parent link="base_link" />
-    <child link="base_footprint" />
-    <origin xyz="0.0 0.26 0" rpy="0 0 0" />
-  </joint>
-  <link name="FrontPivot_Link">
-    <inertial>
-      <origin
-        xyz="0.00350625991709064 0 0"
-        rpy="0 0 0" />
-      <mass
-        value="0.636763996187421" />
-      <inertia
-        ixx="0.000522373966033037"
-        ixy="6.88842321153043E-11"
-        ixz="-2.55687287488004E-10"
-        iyy="0.000692728712644784"
-        iyz="1.31394242797586E-12"
-        izz="0.000643891365515844" />
-    </inertial>
-    <visual>
-      <origin xyz="0 -0.06 0" rpy="0 1.57 0" />
-      <geometry>
-        <!-- <mesh filename="package://segwayrmp_description/meshes/zhuanxiangjia_Link.stl" /> -->
-        <cylinder radius="0.07" length="0.44"/>
-      </geometry>
-      <material name="">
-        <color rgba="0.792156862745098 0.819607843137255 0.933333333333333 1" />
-      </material>
-    </visual>
-    <collision>
-      <origin xyz="0 -0.06 0" rpy="0 1.57 0" />
-      <geometry>
-        <!-- <mesh filename="package://segwayrmp_description/meshes/zhuanxiangjia_Link.stl" /> -->
-        <cylinder radius="0.07" length="0.44"/>
-      </geometry>
-    </collision>
-  </link>
-  <joint name="FrontPivot_joint" type="revolute">
+        <box size="${base_length} ${base_width} ${base_height}" />
+      </geometry>
+    </collision>
+  </link>
+  <!-- Sensors -->
+  <xacro:segwayrmp_laser parent_prefix="base_link" frame_prefix="laser">
+    <origin xyz="0 0.46 0.26" rpy="0 0 0" />
+  </xacro:segwayrmp_laser>
+  <xacro:segwayrmp_imu parent_prefix="base_link" frame_prefix="imu">
+    <origin xyz="0 0 0.14" rpy="0 0 0" />
+  </xacro:segwayrmp_imu>
+  <!-- Steering -->
+  <link name="steering_wheel_link">
+    <inertial>
+      <origin
+        xyz="0 0 0"
+        rpy="0 0 0" />
+      <mass
+        value="0.001" />
+      <inertia ixx="0.00001" ixy="0" ixz="0" iyy="0.00001" iyz="0" izz="0.00001" />
+    </inertial>
+  </link>
+  <joint name="steering_wheel_joint" type="revolute">
     <origin xyz="0 0.46 0.15" rpy="1.5708 0 0" />
     <parent link="base_link" />
-    <child link="FrontPivot_Link" />
+    <child link="steering_wheel_link" />
     <axis xyz="0 -1 0" />
-    <limit
-      lower="-0.36"
-      upper="0.36"
-      effort="0"
-      velocity="0" />
-  </joint>
-  <link
-    name="LeftFrontWheel_Link">
-    <inertial>
-      <origin
-        xyz="-0.175 0 0"
+    <limit lower="-0.36" upper="0.36" effort="0" velocity="1.0" />
+    <dynamics damping="1.0" friction="2.0" />
+  </joint>
+  <link name="front_left_steering_link">
+    <inertial>
+      <origin
+        xyz="-0.1715 0 0"
+        rpy="0 0 0" />
+      <mass
+        value="0.001" />
+      <inertia ixx="0.00001" ixy="0" ixz="0" iyy="0.00001" iyz="0" izz="0.00001" />
+    </inertial>
+  </link>
+  <joint name="front_left_steering_joint" type="revolute">
+    <origin
+      xyz="-0.092435 -0.06 0"
+      rpy="2.9877 0 0" />
+    <parent link="steering_wheel_link" />
+    <child link="front_left_steering_link" />
+    <axis xyz="0 1 0" />
+    <limit lower="-0.36" upper="0.36" effort="1" velocity="1.0" />
+    <dynamics damping="1.0" friction="2.0" />
+  </joint>
+  <link name="front_right_steering_link">
+    <inertial>
+      <origin
+        xyz="-0.17 0 0"
+        rpy="0 0 0" />
+      <mass
+        value="0.001" />
+      <inertia ixx="0.00001" ixy="0" ixz="0" iyy="0.00001" iyz="0" izz="0.00001" />
+    </inertial>
+  </link>
+  <joint name="front_right_steering_joint" type="revolute">
+    <origin
+      xyz="0.099447 -0.06 0"
+      rpy="-1.6671 0 3.1416" />
+    <parent link="steering_wheel_link" />
+    <child link="front_right_steering_link" />
+    <axis xyz="0 0 1" />
+    <limit lower="-0.36" upper="0.36" effort="1" velocity="1.0" />
+    <dynamics damping="1.0" friction="2.0" />
+  </joint>
+  <!-- Wheels -->
+  <link name="front_left_wheel_link">
+    <inertial>
+      <origin
+        xyz="-0.17 0 0"
         rpy="0 0 0" />
       <mass
@@ -118,44 +128,34 @@
         rpy="0 1.57 0" />
       <geometry>
-        <!-- <mesh filename="package://segwayrmp_description/meshes/zuohoulun_Link.stl" /> -->
-        <cylinder radius="0.1" length="0.05"/>
-      </geometry>
-      <material
-        name="">
-        <color
-          rgba="0.792156862745098 0.819607843137255 0.933333333333333 1" />
-      </material>
-    </visual>
-    <collision>
-      <origin
-        xyz="-0.165 0 0"
-        rpy="0 1.57 0" />
-      <geometry>
-        <!-- <mesh filename="package://segwayrmp_description/meshes/zuohoulun_Link.stl" /> -->
-        <cylinder radius="0.1" length="0.05"/>
-      </geometry>
-    </collision>
-  </link>
-  <joint
-    name="LeftFrontWheel_joint"
-    type="continuous">
-    <origin
-      xyz="-0.092435 -0.06 0"
+        <cylinder radius="${wheel_radius}" length="${wheel_length}" />
+      </geometry>
+      <material name="">
+        <color rgba="0.792156862745098 0.819607843137255 0.933333333333333 1" />
+      </material>
+    </visual>
+    <collision>
+      <origin
+        xyz="-0.165 0 0"
+        rpy="0 1.57 0" />
+      <geometry>
+        <cylinder radius="${wheel_radius}" length="${wheel_length}" />
+      </geometry>
+    </collision>
+  </link>
+  <joint name="front_left_wheel_joint" type="continuous">
+    <origin
+      xyz="0 0 0"
       rpy="2.9877 0 0" />
-    <parent
-      link="FrontPivot_Link" />
-    <child
-      link="LeftFrontWheel_Link" />
-    <axis
-      xyz="1 0 0" />
-  </joint>
-  <link
-    name="RightFrontWheel_Link">
-    <inertial>
-      <origin
-        xyz="-0.175 0.01 0"
-        rpy="0 0 0" />
-      <mass
-        value="0.37912408551256" />
+    <parent link="front_left_steering_link" />
+    <child link="front_left_wheel_link" />
+    <axis xyz="1 0 0" />
+    <dynamics damping="1.0" friction="2.0" />
+  </joint>
+  <link name="front_right_wheel_link">
+    <inertial>
+      <origin
+        xyz="0.17 0 0"
+        rpy="0 1.57 0" />
+      <mass value="0.37912408551256" />
       <inertia
         ixx="0.0013562336762928"
@@ -168,47 +168,37 @@
     <visual>
       <origin
-        xyz="-0.165 0 0"
-        rpy="0 1.57 0" />
-      <geometry>
-        <!-- <mesh filename="package://segwayrmp_description/meshes/zuohoulun_Link.stl" /> -->
-        <cylinder radius="0.1" length="0.05"/>
-      </geometry>
-      <material
-        name="">
-        <color
-          rgba="0.792156862745098 0.819607843137255 0.933333333333333 1" />
-      </material>
-    </visual>
-    <collision>
-      <origin
-        xyz="-0.165 0 0"
-        rpy="0 1.57 0" />
-      <geometry>
-        <!-- <mesh filename="package://segwayrmp_description/meshes/zuohoulun_Link.stl" /> -->
-        <cylinder radius="0.1" length="0.05"/>
-      </geometry>
-    </collision>
-  </link>
-  <joint
-    name="RightFrontWheel_joint"
-    type="continuous">
-    <origin
-      xyz="0.099447 -0.06 0"
+        xyz="0.165 0 0"
+        rpy="0 1.57 0" />
+      <geometry>
+        <cylinder radius="${wheel_radius}" length="${wheel_length}" />
+      </geometry>
+      <material name="">
+        <color rgba="0.792156862745098 0.819607843137255 0.933333333333333 1" />
+      </material>
+    </visual>
+    <collision>
+      <origin
+        xyz="0.165 0 0"
+        rpy="0 1.57 0" />
+      <geometry>
+        <cylinder radius="${wheel_radius}" length="${wheel_length}" />
+      </geometry>
+    </collision>
+  </link>
+  <joint name="front_right_wheel_joint" type="continuous">
+    <origin
+      xyz="0 0 0"
       rpy="-1.6671 0 3.1416" />
-    <parent
-      link="FrontPivot_Link" />
-    <child
-      link="RightFrontWheel_Link" />
-    <axis
-      xyz="1 0 0" />
-  </joint>
-  <link
-    name="LeftRearWheel_Link">
+    <parent link="front_right_steering_link" />
+    <child link="front_right_wheel_link" />
+    <axis xyz="1 0 0" />
+    <dynamics damping="1.0" friction="2.0" />
+  </joint>
+  <link name="rear_left_wheel_link">
     <inertial>
       <origin
         xyz="-0.175 4.72112875317676E-05 9.00201436271342E-06"
         rpy="0 0 0" />
-      <mass
-        value="0.634779873374433" />
+      <mass value="0.634779873374433" />
       <inertia
         ixx="0.00181854534335576"
@@ -224,44 +214,34 @@
         rpy="0 1.57 0" />
       <geometry>
-        <!-- <mesh filename="package://segwayrmp_description/meshes/zuohoulun_Link.stl" /> -->
-        <cylinder radius="0.1" length="0.05"/>
-      </geometry>
-      <material
-        name="">
-        <color
-          rgba="0.792156862745098 0.819607843137255 0.933333333333333 1" />
-      </material>
-    </visual>
-    <collision>
-      <origin
-        xyz="-0.165 0 0"
-        rpy="0 1.57 0" />
-      <geometry>
-        <!-- <mesh filename="package://segwayrmp_description/meshes/zuohoulun_Link.stl" /> -->
-        <cylinder radius="0.1" length="0.05"/>
-      </geometry>
-    </collision>
-  </link>
-  <joint
-    name="LeftRearWheel_joint"
-    type="continuous">
+        <cylinder radius="${wheel_radius}" length="${wheel_length}" />
+      </geometry>
+      <material name="">
+        <color rgba="0.792156862745098 0.819607843137255 0.933333333333333 1" />
+      </material>
+    </visual>
+    <collision>
+      <origin
+        xyz="-0.165 0 0"
+        rpy="0 1.57 0" />
+      <geometry>
+        <cylinder radius="${wheel_radius}" length="${wheel_length}" />
+      </geometry>
+    </collision>
+  </link>
+  <joint name="rear_left_wheel_joint" type="continuous">
     <origin
       xyz="-0.1 0.01 0.09"
       rpy="1.5708 0 0" />
-    <parent
-      link="base_link" />
-    <child
-      link="LeftRearWheel_Link" />
-    <axis
-      xyz="1 0 0" />
-  </joint>
-  <link
-    name="RightRearWheel_Link">
+    <parent link="base_link" />
+    <child link="rear_left_wheel_link" />
+    <axis xyz="1 0 0" />
+    <dynamics damping="1.0" friction="2.0" />
+  </joint>
+  <link name="rear_right_wheel_link">
     <inertial>
       <origin
         xyz="-0.175 4.72492608288855E-05 9.01686700283122E-06"
         rpy="0 0 0" />
-      <mass
-        value="0.634778552429949" />
+      <mass value="0.634778552429949" />
       <inertia
         ixx="0.00181854505148151"
@@ -277,137 +257,27 @@
         rpy="0 1.57 0" />
       <geometry>
-        <!-- <mesh filename="package://segwayrmp_description/meshes/zuohoulun_Link.stl" /> -->
-        <cylinder radius="0.1" length="0.05"/>
-      </geometry>
-      <material
-        name="">
-        <color
-          rgba="0.792156862745098 0.819607843137255 0.933333333333333 1" />
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
File: src/segwayrmp_description/urdf/segwayrmp_steering.xacro (robot description, xacro)
@@ -1,111 +1,113 @@
 <?xml version="1.0"?>
 <robot name="segwayrmp_steering" xmlns:xacro="http://ros.org/wiki/xacro">
-    <xacro:macro name="segwayrmp_steering" params="parent_prefix wheel_prefix *joint_pose">
-        <link name="${wheel_prefix}">
-            <inertial>
-              <mass value="0.25" />
-              <inertia ixx="0.00525" ixy="0" ixz="0" iyy="0.00035" iyz="0" izz="0.00525" />
-              <origin xyz="0 0 0" />
-            </inertial>
-            <visual>
-                <origin xyz="0 0 0" rpy="0 0 0" />
-                <geometry>
-                  <cylinder length="0.0001" radius="0.0001" />
-                </geometry>
-            </visual>
-            <collision>
-              <origin xyz="0 ${wheel_length/2} 0" rpy="1.57 0 0" />
-              <geometry>
-                  <cylinder length="${wheel_length}" radius="${wheel_radius-0.01}" />
-              </geometry>
-            </collision>
-        </link>
-        <joint name="${wheel_prefix}_wheel" type="revolute">
-            <parent link="${parent_prefix}"/>
-            <child link="${wheel_prefix}"/>
-            <xacro:insert_block name="joint_pose"/>
-            <axis xyz="0 0 1" />
-            <limit lower="-0.523598767" upper="0.523598767" effort="5" velocity="0.5" />
-            <dynamics damping="1.0" friction="2.0"/>
-        </joint>
-        <link name="front_left_wheel_link">
-          <inertial>
-            <mass value="0.25" />
-            <inertia ixx="0.00525" ixy="0" ixz="0" iyy="0.00035" iyz="0" izz="0.00525" />
-            <origin xyz="0 0 0" />
-          </inertial>
-          <visual>
-              <origin xyz="0 0 0" rpy="0 0 0" />
-              <geometry>
-                  <mesh filename="file://$(find segwayrmp_description)/meshes/segwayrmp_wheel.dae" />
-              </geometry>
-          </visual>
-          <collision>
-            <origin xyz="0 ${wheel_length/2} 0" rpy="1.57 0 0" />
-            <geometry>
-                <cylinder length="${wheel_length}" radius="${wheel_radius}" />
-            </geometry>
-          </collision>
-      </link>
-      <joint name="front_left_wheel" type="continuous">
-          <parent link="${wheel_prefix}"/>
-          <child link="front_left_wheel_link"/>
-          <origin xyz="0 0 0" rpy="0 0  0" />
-          <axis xyz="0 1 0"/>
-      </joint>
-    </xacro:macro>
-    <xacro:macro name="segwayrmp_right_steering_hinge" params="parent_prefix wheel_prefix *joint_pose">
-        <link name="${wheel_prefix}">
-          <inertial>
-            <mass value="0.25" />
-            <inertia ixx="0.00525" ixy="0" ixz="0" iyy="0.00035" iyz="0" izz="0.00525" />
-            <origin xyz="0 0 0" />
-          </inertial>
-            <visual>
-                <origin xyz="0 0 0" rpy="0 0 0" />
-                <geometry>
-                  <cylinder length="0.0001" radius="0.0001" />
-                </geometry>
-            </visual>
-            <collision>
-              <origin xyz="0 ${wheel_length/2} 0" rpy="1.57 0 0" />
-              <geometry>
-                  <cylinder length="${wheel_length}" radius="${wheel_radius-0.01}" />
-              </geometry>
-            </collision>
-        </link>
-        <joint name="${wheel_prefix}_wheel" type="revolute">
-            <parent link="${parent_prefix}"/>
-            <child link="${wheel_prefix}"/>
-            <xacro:insert_block name="joint_pose"/>
-            <axis xyz="0 0 -1"/>
-            <limit lower="-0.523598767" upper="0.523598767" effort="5" velocity="0.5" />
-            <dynamics damping="1.0" friction="2.0"/>
-        </joint>
-        <link name="front_right_wheel_link">
-          <inertial>
-            <mass value="0.25" />
-            <inertia ixx="0.00525" ixy="0" ixz="0" iyy="0.00035" iyz="0" izz="0.00525" />
-            <origin xyz="0 0 0" />
-          </inertial>
-          <visual>
-              <origin xyz="0 0 0" rpy="0 0 0" />
-              <geometry>
-                  <mesh filename="file://$(find segwayrmp_description)/meshes/segwayrmp_wheel.dae" />
-              </geometry>
-          </visual>
-          <collision>
-            <origin xyz="0 ${wheel_length/2} 0" rpy="1.57 0 0" />
-            <geometry>
-                <cylinder length="${wheel_length}" radius="${wheel_radius}" />
-            </geometry>
-          </collision>
-      </link>
-      <joint name="front_right_wheel" type="continuous">
-          <parent link="${wheel_prefix}"/>
-          <child link="front_right_wheel_link"/>
-          <origin xyz="0 0 0" rpy="0 0  0" />
-          <axis xyz="0 -1 0"/>
-      </joint>
-    </xacro:macro>
+  <xacro:macro name="segwayrmp_steering" params="parent_prefix wheel_prefix *joint_pose">
+    <link name="${wheel_prefix}">
+      <inertial>
+        <mass value="0.25" />
+        <inertia ixx="0.00525" ixy="0" ixz="0" iyy="0.00035" iyz="0" izz="0.00525" />
+        <origin xyz="0 0 0" />
+      </inertial>
+      <visual>
+        <origin xyz="0 0 0" rpy="0 0 0" />
+        <geometry>
+          <cylinder length="0.0001" radius="0.0001" />
+        </geometry>
+      </visual>
+      <collision>
+        <origin xyz="0 ${wheel_length/2} 0" rpy="1.57 0 0" />
+        <geometry>
+          <cylinder length="${wheel_length}" radius="${wheel_radius-0.01}" />
+        </geometry>
+      </collision>
+    </link>
+    <joint name="${wheel_prefix}_wheel" type="revolute">
+      <parent link="${parent_prefix}" />
+      <child link="${wheel_prefix}" />
+      <xacro:insert_block name="joint_pose" />
+      <axis xyz="0 0 1" />
+      <limit lower="-0.523598767" upper="0.523598767" effort="5" velocity="0.5" />
+      <dynamics damping="1.0" friction="2.0" />
+    </joint>
+    <link name="front_left_wheel_link">
+      <inertial>
+        <mass value="0.25" />
+        <inertia ixx="0.00525" ixy="0" ixz="0" iyy="0.00035" iyz="0" izz="0.00525" />
+        <origin xyz="0 0 0" />
+      </inertial>
+      <visual>
+        <origin xyz="0 0 0" rpy="0 0 0" />
+        <geometry>
+          <!-- <mesh filename="file://$(find segwayrmp_description)/meshes/segwayrmp_wheel.dae" /> -->
+          <cylinder radius="0.1" length="0.05" />
+        </geometry>
+      </visual>
+      <collision>
+        <origin xyz="0 ${wheel_length/2} 0" rpy="1.57 0 0" />
+        <geometry>
+          <cylinder length="${wheel_length}" radius="${wheel_radius}" />
+        </geometry>
+      </collision>
+    </link>
+    <joint name="front_left_wheel" type="continuous">
+      <parent link="${wheel_prefix}" />
+      <child link="front_left_wheel_link" />
+      <origin xyz="0 0 0" rpy="0 0  0" />
+      <axis xyz="0 1 0" />
+    </joint>
+  </xacro:macro>
+  <xacro:macro name="segwayrmp_right_steering_hinge" params="parent_prefix wheel_prefix *joint_pose">
+    <link name="${wheel_prefix}">
+      <inertial>
+        <mass value="0.25" />
+        <inertia ixx="0.00525" ixy="0" ixz="0" iyy="0.00035" iyz="0" izz="0.00525" />
+        <origin xyz="0 0 0" />
+      </inertial>
+      <visual>
+        <origin xyz="0 0 0" rpy="0 0 0" />
+        <geometry>
+          <cylinder length="0.0001" radius="0.0001" />
+        </geometry>
+      </visual>
+      <collision>
+        <origin xyz="0 ${wheel_length/2} 0" rpy="1.57 0 0" />
+        <geometry>
+          <cylinder length="${wheel_length}" radius="${wheel_radius-0.01}" />
+        </geometry>
+      </collision>
+    </link>
+    <joint name="${wheel_prefix}_wheel" type="continuous">
+      <parent link="${parent_prefix}" />
+      <child link="${wheel_prefix}" />
+      <xacro:insert_block name="joint_pose" />
+      <axis xyz="1 0 0" />
+      <!-- <limit lower="-0.523598767" upper="0.523598767" effort="5" velocity="0.5" /> -->
+      <dynamics damping="1.0" friction="2.0" />
+    </joint>
+    <link name="front_right_wheel_link">
+      <inertial>
+        <mass value="0.25" />
+        <inertia ixx="0.00525" ixy="0" ixz="0" iyy="0.00035" iyz="0" izz="0.00525" />
+        <origin xyz="0 0 0" />
+      </inertial>
+      <visual>
+        <origin xyz="0 0 0" rpy="0 0 0" />
+        <geometry>
+          <!-- <mesh filename="file://$(find segwayrmp_description)/meshes/segwayrmp_wheel.dae" /> -->
+          <cylinder radius="0.1" length="0.05" />
+        </geometry>
+      </visual>
+      <collision>
+        <origin xyz="0 ${wheel_length/2} 0" rpy="1.57 0 0" />
+        <geometry>
+          <cylinder length="${wheel_length}" radius="${wheel_radius}" />
+        </geometry>
+      </collision>
+    </link>
+    <joint name="front_right_wheel" type="continuous">
+      <parent link="${wheel_prefix}" />
+      <child link="front_right_wheel_link" />
+      <origin xyz="0 0 0" rpy="0 0  0" />
+      <axis xyz="0 -1 0" />
+    </joint>
+  </xacro:macro>
 </robot>
