Commit message: Update default_value for joint_state_publisher_gui to false and adjusted urdf.xacro values

File: src/segwayrmp_description/urdf/segwayrmp.urdf.xacro (robot description, xacro)
@@ -19,7 +19,7 @@
     <inertial>
       <origin
-        xyz="0 0.23 0.19"
-        rpy="0 0 0" />
-      <mass value="2.42397545608915" />
+        xyz="0 0.2 0.19"
+        rpy="0 0 0" />
+      <mass value="12.0" />
       <inertia ixx="0.0296962022350776" ixy="0" ixz="0"
         iyy="0.00646533575042488" iyz="0" izz="0.0331663553221158" />
@@ -54,8 +54,22 @@
         xyz="0 0 0"
         rpy="0 0 0" />
-      <mass
-        value="0.001" />
-      <inertia ixx="0.00001" ixy="0" ixz="0" iyy="0.00001" iyz="0" izz="0.00001" />
-    </inertial>
+      <mass value="0.3" />
+      <inertia ixx="0.0008778" ixy="0.0" ixz="0.0" iyy="0.00011879" iyz="0.0" izz="0.0008778" />
+    </inertial>
+    <visual>
+      <origin xyz="0 0 0" rpy="0 0 0" />
+      <geometry>
+        <box size="0.01 0.01 0.01" />
+      </geometry>
+      <material name="">
+        <color rgba="0.792156862745098 0.819607843137255 0.933333333333333 1" />
+      </material>
+    </visual>
+    <collision>
+      <origin xyz="0 0 0" rpy="0 0 0" />
+      <geometry>
+        <box size="0.01 0.01 0.01" />
+      </geometry>
+    </collision>
   </link>
   <joint name="steering_wheel_joint" type="revolute">
@@ -63,47 +77,40 @@
     <parent link="base_link" />
     <child link="steering_wheel_link" />
-    <axis xyz="0 -1 0" />
-    <limit lower="-0.36" upper="0.36" effort="0" velocity="1.0" />
-    <dynamics damping="1.0" friction="2.0" />
-  </joint>
-  <link name="front_left_steering_link">
-    <inertial>
-      <origin
-        xyz="-0.1715 0 0"
-        rpy="0 0 0" />
-      <mass
-        value="0.001" />
-      <inertia ixx="0.00001" ixy="0" ixz="0" iyy="0.00001" iyz="0" izz="0.00001" />
-    </inertial>
-  </link>
-  <joint name="front_left_steering_joint" type="revolute">
-    <origin
-      xyz="-0.092435 -0.06 0"
-      rpy="2.9877 0 0" />
+    <axis xyz="0 1 0" />
+    <limit lower="-0.36" upper="0.36" effort="5" velocity="1.0" />
+    <dynamics damping="0.1" friction="1.0" />
+  </joint>
+  <link name="front_wheels_link">
+    <inertial>
+      <origin
+        xyz="0 0 0"
+        rpy="0 0 1.57" />
+      <mass value="0.379124506048444" />
+      <inertia ixx="0.00001697" ixy="0.0" ixz="0.0" iyy="0.01254" iyz="0.0" izz="0.01254" />
+    </inertial>
+    <visual>
+      <origin xyz="0 0 0" rpy="0 1.57 0" />
+      <geometry>
+        <cylinder radius="0.07" length="0.45" />
+      </geometry>
+      <material name="">
+        <color rgba="0.792156862745098 0.819607843137255 0.933333333333333 1" />
+      </material>
+    </visual>
+    <collision>
+      <origin xyz="0 0 0" rpy="0 1.57 0" />
+      <geometry>
+        <cylinder radius="0.07" length="0.45" />
+      </geometry>
+    </collision>
+  </link>
+  <joint name="front_wheels_joint" type="continuous">
+    <origin
+      xyz="0 -0.06 0"
+      rpy="0 0 0" />
     <parent link="steering_wheel_link" />
-    <child link="front_left_steering_link" />
-    <axis xyz="0 1 0" />
-    <limit lower="-0.36" upper="0.36" effort="1" velocity="1.0" />
-    <dynamics damping="1.0" friction="2.0" />
-  </joint>
-  <link name="front_right_steering_link">
-    <inertial>
-      <origin
-        xyz="-0.17 0 0"
-        rpy="0 0 0" />
-      <mass
-        value="0.001" />
-      <inertia ixx="0.00001" ixy="0" ixz="0" iyy="0.00001" iyz="0" izz="0.00001" />
-    </inertial>
-  </link>
-  <joint name="front_right_steering_joint" type="revolute">
-    <origin
-      xyz="0.099447 -0.06 0"
-      rpy="-1.6671 0 3.1416" />
-    <parent link="steering_wheel_link" />
-    <child link="front_right_steering_link" />
-    <axis xyz="0 0 1" />
-    <limit lower="-0.36" upper="0.36" effort="1" velocity="1.0" />
-    <dynamics damping="1.0" friction="2.0" />
+    <child link="front_wheels_link" />
+    <axis xyz="-1 0 0" />
+    <dynamics damping="0.1" friction="1.0" />
   </joint>
   <!-- Wheels -->
@@ -111,58 +118,57 @@
     <inertial>
       <origin
-        xyz="-0.17 0 0"
-        rpy="0 0 0" />
-      <mass
-        value="0.379124506048444" />
-      <inertia
-        ixx="0.00135623331658277"
-        ixy="-2.05858146537997E-08"
-        ixz="2.75425144310775E-07"
-        iyy="0.00074553860560749"
-        iyz="-2.05160697747808E-08"
-        izz="0.000744863292198173" />
-    </inertial>
-    <visual>
-      <origin
-        xyz="-0.165 0 0"
-        rpy="0 1.57 0" />
-      <geometry>
-        <cylinder radius="${wheel_radius}" length="${wheel_length}" />
-      </geometry>
-      <material name="">
-        <color rgba="0.792156862745098 0.819607843137255 0.933333333333333 1" />
-      </material>
-    </visual>
-    <collision>
-      <origin
-        xyz="-0.165 0 0"
-        rpy="0 1.57 0" />
-      <geometry>
-        <cylinder radius="${wheel_radius}" length="${wheel_length}" />
-      </geometry>
-    </collision>
-  </link>
-  <joint name="front_left_wheel_joint" type="continuous">
-    <origin
-      xyz="0 0 0"
-      rpy="2.9877 0 0" />
-    <parent link="front_left_steering_link" />
+        xyz="-0.175 0 0"
+        rpy="0 0 0" />
+      <mass value="0.379124506048444" />
+      <inertia
+        ixx="0.00135623331658277"
+        ixy="-2.05858146537997E-08"
+        ixz="2.75425144310775E-07"
+        iyy="0.00074553860560749"
+        iyz="-2.05160697747808E-08"
+        izz="0.000744863292198173" />
+    </inertial>
+    <visual>
+      <origin
+        xyz="-0.165 0 0"
+        rpy="0 1.57 0" />
+      <geometry>
+        <cylinder radius="${wheel_radius}" length="${wheel_length}" />
+      </geometry>
+      <material name="">
+        <color rgba="0.792156862745098 0.819607843137255 0.933333333333333 1" />
+      </material>
+    </visual>
+    <collision>
+      <origin
+        xyz="-0.165 0 0"
+        rpy="0 1.57 0" />
+      <geometry>
+        <cylinder radius="${wheel_radius}" length="${wheel_length}" />
+      </geometry>
+    </collision>
+  </link>
+  <joint name="front_left_wheel_joint" type="fixed">
+    <origin
+      xyz="-0.1 0 0"
+      rpy="3.14 0 0" />
+    <parent link="front_wheels_link" />
     <child link="front_left_wheel_link" />
-    <axis xyz="1 0 0" />
-    <dynamics damping="1.0" friction="2.0" />
+    <!-- <axis xyz="1 0 0" /> -->
+    <dynamics damping="0.1" friction="1.0" />
   </joint>
   <link name="front_right_wheel_link">
     <inertial>
       <origin
-        xyz="0.17 0 0"
-        rpy="0 1.57 0" />
-      <mass value="0.37912408551256" />
-      <inertia
-        ixx="0.0013562336762928"
-        ixy="-2.05946493125457E-08"
-        ixz="2.75615782692675E-07"
-        iyy="0.0007455386716045"
-        iyz="-2.12571382999838E-08"
-        izz="0.000744862395561634" />
+        xyz="0.175 0 0"
+        rpy="0 1.57 0" />
+      <mass value="0.379124506048444" />
+      <inertia
+        ixx="0.00135623331658277"
+        ixy="-2.05858146537997E-08"
+        ixz="2.75425144310775E-07"
+        iyy="0.00074553860560749"
+        iyz="-2.05160697747808E-08"
+        izz="0.000744863292198173" />
     </inertial>
     <visual>
@@ -186,12 +192,12 @@
     </collision>
   </link>
-  <joint name="front_right_wheel_joint" type="continuous">
-    <origin
-      xyz="0 0 0"
-      rpy="-1.6671 0 3.1416" />
-    <parent link="front_right_steering_link" />
+  <joint name="front_right_wheel_joint" type="fixed">
+    <origin
+      xyz="0.1 0 0"
+      rpy="1.57 3.1416 3.1416" />
+    <parent link="front_wheels_link" />
     <child link="front_right_wheel_link" />
-    <axis xyz="1 0 0" />
-    <dynamics damping="1.0" friction="2.0" />
+    <!-- <axis xyz="1 0 0" /> -->
+    <dynamics damping="0.1" friction="1.0" />
   </joint>
   <link name="rear_left_wheel_link">
@@ -200,12 +206,12 @@
         xyz="-0.175 4.72112875317676E-05 9.00201436271342E-06"
         rpy="0 0 0" />
-      <mass value="0.634779873374433" />
-      <inertia
-        ixx="0.00181854534335576"
-        ixy="3.33041385279325E-07"
-        ixz="-2.8378478388468E-07"
-        iyy="0.00101390067982028"
-        iyz="-5.2299696505564E-09"
-        izz="0.00101270577373137" />
+      <mass value="0.379124506048444" />
+      <inertia
+        ixx="0.00135623331658277"
+        ixy="-2.05858146537997E-08"
+        ixz="2.75425144310775E-07"
+        iyy="0.00074553860560749"
+        iyz="-2.05160697747808E-08"
+        izz="0.000744863292198173" />
     </inertial>
     <visual>
@@ -235,6 +241,6 @@
     <parent link="base_link" />
     <child link="rear_left_wheel_link" />
-    <axis xyz="1 0 0" />
-    <dynamics damping="1.0" friction="2.0" />
+    <axis xyz="-1 0 0" />
+    <dynamics damping="0.1" friction="1.0" />
   </joint>
   <link name="rear_right_wheel_link">
@@ -243,12 +249,12 @@
         xyz="-0.175 4.72492608288855E-05 9.01686700283122E-06"
         rpy="0 0 0" />
-      <mass value="0.634778552429949" />
-      <inertia
-        ixx="0.00181854505148151"
-        ixy="3.32515010548019E-07"
-        ixz="-2.83394847813244E-07"
-        iyy="0.00101390105479182"
-        iyz="-5.03852728516005E-09"
-        izz="0.00101270465329001" />
+      <mass value="0.379124506048444" />
+      <inertia
+        ixx="0.00135623331658277"
+        ixy="-2.05858146537997E-08"
+        ixz="2.75425144310775E-07"
+        iyy="0.00074553860560749"
+        iyz="-2.05160697747808E-08"
+        izz="0.000744863292198173" />
     </inertial>
     <visual>
@@ -275,9 +281,9 @@
     <origin
       xyz="0.1 0.01 0.09"
-      rpy="0.17453 0 -3.1416" />
+      rpy="0 0 3.1416" />
     <parent link="base_link" />
     <child link="rear_right_wheel_link" />
     <axis xyz="1 0 0" />
-    <dynamics damping="1.0" friction="2.0" />
+    <dynamics damping="0.1" friction="1.0" />
   </joint>
 </robot>

File: src/segwayrmp_description/urdf/segwayrmp_steering.xacro (robot description, xacro)
@@ -1,9 +1,47 @@
 <?xml version="1.0"?>
 <robot name="segwayrmp_steering" xmlns:xacro="http://ros.org/wiki/xacro">
-  <xacro:macro name="segwayrmp_steering" params="parent_prefix wheel_prefix *joint_pose">
-    <link name="${wheel_prefix}">
+  <xacro:macro name="segwayrmp_steering" params="parent_prefix steering_prefix *joint_pose">
+    <link name="${steering_prefix}">
       <inertial>
-        <mass value="0.25" />
-        <inertia ixx="0.00525" ixy="0" ixz="0" iyy="0.00035" iyz="0" izz="0.00525" />
+        <origin
+          xyz="0 0 0"
+          rpy="0 0 0" />
+        <mass value="0.3" />
+        <inertia ixx="0.0008778" ixy="0.0" ixz="0.0" iyy="0.00011879" iyz="0.0" izz="0.0008778" />
+      </inertial>
+      <visual>
+        <origin xyz="0 0 0" rpy="0 0 0" />
+        <geometry>
+          <box size="0.01 0.01 0.01" />
+        </geometry>
+        <material name="">
+          <color rgba="0.792156862745098 0.819607843137255 0.933333333333333 1" />
+        </material>
+      </visual>
+      <collision>
+        <origin xyz="0 0 0" rpy="0 0 0" />
+        <geometry>
+          <box size="0.01 0.01 0.01" />
+        </geometry>
+      </collision>
+    </link>
+    <joint name="${steering_prefix}_wheel" type="revolute">
+      <parent link="${parent_prefix}" />
+      <child link="${steering_prefix}" />
+      <xacro:insert_block name="joint_pose" />
+      <axis xyz="0 1 0" />
+      <limit lower="-0.36" upper="0.36" effort="5" velocity="1.0" />
+      <dynamics damping="1.0" friction="1.0" />
+    </joint>
+    <link name="front_left_wheel_link">
+      <inertial>
+        <mass value="0.379124506048444" />
+        <inertia
+          ixx="0.00135623331658277"
+          ixy="-2.05858146537997E-08"
+          ixz="2.75425144310775E-07"
+          iyy="0.00074553860560749"
+          iyz="-2.05160697747808E-08"
+          izz="0.000744863292198173" />
         <origin xyz="0 0 0" />
       </inertial>
@@ -11,39 +49,11 @@
         <origin xyz="0 0 0" rpy="0 0 0" />
         <geometry>
-          <cylinder length="0.0001" radius="0.0001" />
+          <cylinder radius="${wheel_radius}" length="${wheel_length}" />
         </geometry>
       </visual>
       <collision>
-        <origin xyz="0 ${wheel_length/2} 0" rpy="1.57 0 0" />
+        <origin xyz="0 0 0" rpy="1.57 0 0" />
         <geometry>
-          <cylinder length="${wheel_length}" radius="${wheel_radius-0.01}" />
-        </geometry>
-      </collision>
-    </link>
-    <joint name="${wheel_prefix}_wheel" type="revolute">
-      <parent link="${parent_prefix}" />
-      <child link="${wheel_prefix}" />
-      <xacro:insert_block name="joint_pose" />
-      <axis xyz="0 0 1" />
-      <limit lower="-0.523598767" upper="0.523598767" effort="5" velocity="0.5" />
-      <dynamics damping="1.0" friction="2.0" />
-    </joint>
-    <link name="front_left_wheel_link">
-      <inertial>
-        <mass value="0.25" />
-        <inertia ixx="0.00525" ixy="0" ixz="0" iyy="0.00035" iyz="0" izz="0.00525" />
-        <origin xyz="0 0 0" />
-      </inertial>
-      <visual>
-        <origin xyz="0 0 0" rpy="0 0 0" />
-        <geometry>
-          <!-- <mesh filename="file://$(find segwayrmp_description)/meshes/segwayrmp_wheel.dae" /> -->
-          <cylinder radius="0.1" length="0.05" />
-        </geometry>
-      </visual>
-      <collision>
-        <origin xyz="0 ${wheel_length/2} 0" rpy="1.57 0 0" />
-        <geometry>
-          <cylinder length="${wheel_length}" radius="${wheel_radius}" />
+          <cylinder radius="${wheel_radius}" length="${wheel_length}" />
         </geometry>
       </collision>
@@ -53,5 +63,5 @@
       <child link="front_left_wheel_link" />
       <origin xyz="0 0 0" rpy="0 0  0" />
-      <axis xyz="0 1 0" />
+      <axis xyz="1 0 0" />
     </joint>
   </xacro:macro>
@@ -81,11 +91,16 @@
       <xacro:insert_block name="joint_pose" />
       <axis xyz="1 0 0" />
-      <!-- <limit lower="-0.523598767" upper="0.523598767" effort="5" velocity="0.5" /> -->
-      <dynamics damping="1.0" friction="2.0" />
+      <dynamics damping="1.0" friction="1.0" />
     </joint>
     <link name="front_right_wheel_link">
       <inertial>
-        <mass value="0.25" />
-        <inertia ixx="0.00525" ixy="0" ixz="0" iyy="0.00035" iyz="0" izz="0.00525" />
+        <mass value="0.379124506048444" />
+        <inertia
+          ixx="0.00135623331658277"
+          ixy="-2.05858146537997E-08"
+          ixz="2.75425144310775E-07"
+          iyy="0.00074553860560749"
+          iyz="-2.05160697747808E-08"
+          izz="0.000744863292198173" />
         <origin xyz="0 0 0" />
       </inertial>
@@ -93,12 +108,11 @@
         <origin xyz="0 0 0" rpy="0 0 0" />
         <geometry>
-          <!-- <mesh filename="file://$(find segwayrmp_description)/meshes/segwayrmp_wheel.dae" /> -->
-          <cylinder radius="0.1" length="0.05" />
+          <cylinder radius="${wheel_radius}" length="${wheel_length}" />
         </geometry>
       </visual>
       <collision>
-        <origin xyz="0 ${wheel_length/2} 0" rpy="1.57 0 0" />
+        <origin xyz="0 0 0" rpy="1.57 0 0" />
         <geometry>
-          <cylinder length="${wheel_length}" radius="${wheel_radius}" />
+          <cylinder radius="${wheel_radius}" length="${wheel_length}" />
         </geometry>
       </collision>
@@ -108,5 +122,5 @@
       <child link="front_right_wheel_link" />
       <origin xyz="0 0 0" rpy="0 0  0" />
-      <axis xyz="0 -1 0" />
+      <axis xyz="1 0 0" />
     </joint>
   </xacro:macro>

File: src/segwayrmp_description/urdf/segwayrmp_xacro.xacro (robot description, xacro)
@@ -5,5 +5,5 @@
       <inertial>
         <origin xyz="0 0 0" />
-        <mass value="0.5" />
+        <mass value="0.3" />
         <inertia ixx="0.01055" ixy="0" ixz="0" iyy="0.00075" iyz="0" izz="0.01055" />
       </inertial>
@@ -11,5 +11,5 @@
         <origin xyz="0 0 0" rpy="0 0 0" />
         <geometry>
-          <cylinder radius="0.1" length="0.05" />
+          <cylinder radius="${wheel_length}" length="${wheel_radius}"/>
         </geometry>
       </visual>
@@ -25,5 +25,33 @@
       <child link="${wheel_prefix}_wheel_link" />
       <xacro:insert_block name="joint_pose" />
-      <axis xyz="0 ${reflect*1} 0" />
+      <axis xyz="${reflect*1} 0 0" />
+    </joint>
+  </xacro:macro>
+  <xacro:macro name="segwayrmp_steering" params="parent_prefix steering_prefix *joint_pose">
+    <link name="${steering_prefix}_link">
+      <inertial>
+        <origin xyz="0 0 0" />
+        <mass value="0.3" />
+        <inertia ixx="0.0008778" ixy="0.0" ixz="0.0" iyy="0.00011879" iyz="0.0" izz="0.0008778" />
+      </inertial>
+      <visual>
+        <origin xyz="0 0 0" rpy="0 0 0" />
+        <geometry>
+          <box size="0.01 0.01 0.01" />
+        </geometry>
+      </visual>
+      <collision>
+        <origin xyz="0 0 0" rpy="0 0 0" />
+        <geometry>
+          <box size="0.01 0.01 0.01" />
+        </geometry>
+      </collision>
+    </link>
+    <joint name="${steering_prefix}_joint" type="revolute">
+      <parent link="${parent_prefix}" />
+      <child link="${steering_prefix}_link" />
+      <xacro:insert_block name="joint_pose" />
+      <axis xyz="0 1 0" />
+      <limit lower="-0.36" upper="0.36" effort="0" velocity="1.0" />
     </joint>
   </xacro:macro>
