Commit message: Updated nav2 stack for simulation segwayrmp_navigation_launch.py: remapped /cmd_vel to /tricycle_controller/cmd_vel for simulation

File: src/segwayrmp_description/urdf/segwayrmp.urdf.xacro (robot description, xacro)
@@ -1,289 +1,221 @@
-<?xml version="1.0" encoding="UTF-8"?>
-<!-- This URDF was automatically created by SolidWorks to URDF Exporter! Originally created by
-Stephen Brawner (brawner@gmail.com)
-     Commit Version: 1.5.1-0-g916b5db  Build Version: 1.5.7152.31018
-     For more information, please see http://wiki.ros.org/sw_urdf_exporter -->
-<robot name="segwayrmp_urdf" xmlns:xacro="http://ros.org/wiki/xacro">
-  <xacro:arg name="robot_namespace" default="/" />
-  <xacro:include filename="$(find segwayrmp_description)/urdf/segwayrmp_xacro.xacro" />
-  <!-- <xacro:include filename="$(find segwayrmp_description)/urdf/segwayrmp_steering.xacro" /> -->
-  <xacro:include filename="$(find segwayrmp_description)/urdf/segwayrmp_ackerman.gazebo" />
-  <!-- Define robot constants -->
-  <xacro:property name="base_length" value="0.18" />
-  <xacro:property name="base_width" value="0.61" />
-  <xacro:property name="base_height" value="0.09" />
+<?xml version="1.0"?>
+<robot name="Segwayrmp" xmlns:xacro="http://ros.org/wiki/xacro">
+  <material name="Black">
+    <color rgba="0 0 0 1" />
+  </material>
+  <material name="Grey">
+    <color rgba="0.8 0.8 0.8 1" />
+  </material>
+  <material name="Orange">
+    <color rgba="1 0.6 0 1" />
+  </material>
+  <material name="White">
+    <color rgba="1 1 1 1" />
+  </material>
   <xacro:property name="wheel_length" value="0.05" />
   <xacro:property name="wheel_radius" value="0.1" />
-  <!-- Robot Base -->
-  <link name="base_link">
-    <inertial>
-      <origin
-        xyz="0 0.2 0.19"
-        rpy="0 0 0" />
-      <mass value="12.0" />
-      <inertia ixx="0.0296962022350776" ixy="0" ixz="0"
-        iyy="0.00646533575042488" iyz="0" izz="0.0331663553221158" />
-    </inertial>
-    <visual>
-      <origin xyz="0 0.24 0.21" rpy="0 0 0" />
-      <geometry>
-        <box size="${base_length} ${base_width} ${base_height}" />
-      </geometry>
-      <material name="">
-        <color rgba="0.792156862745098 0.819607843137255 0.933333333333333 1" />
-      </material>
-    </visual>
-    <collision>
-      <origin xyz="0 0.24 0.21" rpy="0 0 0" />
-      <geometry>
-        <box size="${base_length} ${base_width} ${base_height}" />
-      </geometry>
-    </collision>
-  </link>
+  <link name="base_link" />
+  <!-- base_footprint -->
+  <link name="base_footprint">
+    <collision>
+      <origin xyz="0 0 0" rpy="0 0 0" />
+      <geometry>
+        <box size="0.61 0.18 0.09" />
+      </geometry>
+    </collision>
+    <visual>
+      <origin xyz="0 0 0" rpy="0 0 0" />
+      <geometry>
+        <box size="0.61 0.18 0.09" />
+      </geometry>
+      <material name="Orange" />
+    </visual>
+    <inertial>
+      <origin xyz="-0.05 0 0" rpy="0 0 0" />
+      <mass value="16" />
+      <inertia ixx="0.06192" ixy="0" ixz="0" iyy="0.28416" iyz="0" izz="0.318336" />
+    </inertial>
+  </link>
+  <joint name="base_footprint_joint" type="fixed">
+    <origin xyz="0.305 0 0.21" rpy="0 0 0" />
+    <parent link="base_link" />
+    <child link="base_footprint" />
+  </joint>
+  <!-- Left Rear Wheel Link -->
+  <link name="left_rear_wheel">
+    <collision>
+      <geometry>
+        <cylinder length="${wheel_length}" radius="${wheel_radius}" />
+      </geometry>
+    </collision>
+    <visual>
+      <geometry>
+        <cylinder length="${wheel_length}" radius="${wheel_radius}" />
+      </geometry>
+      <material name="Black" />
+    </visual>
+    <inertial>
+      <mass value="1.2" />
+      <inertia ixx="0.00145833" ixy="0.0" ixz="0.0" iyy="0.00145833" iyz="0.0" izz="0.00125" />
+    </inertial>
+  </link>
+  <joint name="left_rear_wheel_joint" type="continuous">
+    <origin xyz="-0.25 0.15 -0.09" rpy="-1.57 0 0" />
+    <parent link="base_footprint" />
+    <child link="left_rear_wheel" />
+    <axis xyz="0 0 1" />
+    <dynamics damping="0.2" />
+  </joint>
+  <!-- Right Rear Wheel Link -->
+  <link name="right_rear_wheel">
+    <collision>
+      <geometry>
+        <cylinder length="${wheel_length}" radius="${wheel_radius}" />
+      </geometry>
+    </collision>
+    <visual>
+      <geometry>
+        <cylinder length="${wheel_length}" radius="${wheel_radius}" />
+      </geometry>
+      <material name="Black" />
+    </visual>
+    <inertial>
+      <mass value="1.2" />
+      <inertia ixx="0.00145833" ixy="0.0" ixz="0.0" iyy="0.00145833" iyz="0.0" izz="0.00125" />
+    </inertial>
+  </link>
+  <joint name="right_rear_wheel_joint" type="continuous">
+    <origin xyz="-0.25 -0.15 -0.09" rpy="-1.57 0 0" />
+    <parent link="base_footprint" />
+    <child link="right_rear_wheel" />
+    <axis xyz="0 0 1" />
+    <dynamics damping="0.2" />
+  </joint>
+  <!-- Steering Link -->
+  <link name="steering_link">
+    <visual>
+      <geometry>
+        <box size="0.01 0.01 0.01" />
+      </geometry>
+      <material name="Black" />
+    </visual>
+    <inertial>
+      <origin xyz="0 0 0" rpy="0 0 0" />
+      <mass value="0.05" />
+      <inertia ixx="0.001" ixy="0.0" ixz="0.0" iyy="0.001" iyz="0.0" izz="0.001" />
+    </inertial>
+  </link>
+  <joint name="steering_joint" type="revolute">
+    <origin xyz="0.25 0 -0.09" rpy="0 0 0" />
+    <parent link="base_footprint" />
+    <child link="steering_link" />
+    <axis xyz="0 0 1" />
+    <limit lower="-0.36" upper="0.36" effort="0.0" velocity="0.0" />
+    <dynamics damping="0.2" />
+  </joint>
+  <!-- Traction Wheel Link -->
+  <link name="front_wheel_link">
+    <collision>
+      <geometry>
+        <cylinder length="${wheel_length}" radius="${wheel_radius}" />
+      </geometry>
+    </collision>
+    <visual>
+      <geometry>
+        <cylinder length="${wheel_length}" radius="${wheel_radius}" />
+      </geometry>
+      <material name="Black" />
+    </visual>
+    <inertial>
+      <origin xyz="0 0 0" rpy="0 0 0" />
+      <mass value="1.2" />
+      <inertia ixx="0.0145833" ixy="0.0" ixz="0.0" iyy="0.0145833" iyz="0.0" izz="0.0125" />
+    </inertial>
+  </link>
+  <joint name="traction_joint" type="continuous">
+    <parent link="steering_link" />
+    <child link="front_wheel_link" />
+    <origin xyz="0 0 0" rpy="-1.57 1.57 0" />
+    <axis xyz="0 0 1" />
+    <dynamics damping="0.2" />
+  </joint>
   <!-- Sensors -->
-  <xacro:segwayrmp_laser parent_prefix="base_link" frame_prefix="laser">
-    <origin xyz="0 0.46 0.26" rpy="0 0 0" />
-  </xacro:segwayrmp_laser>
-  <xacro:segwayrmp_imu parent_prefix="base_link" frame_prefix="imu">
-    <origin xyz="0 0 0.14" rpy="0 0 0" />
-  </xacro:segwayrmp_imu>
-  <!-- Steering -->
-  <link name="steering_wheel_link">
-    <inertial>
-      <origin
-        xyz="0 0 0"
-        rpy="0 0 0" />
-      <mass value="0.3" />
-      <inertia ixx="0.0008778" ixy="0.0" ixz="0.0" iyy="0.00011879" iyz="0.0" izz="0.0008778" />
-    </inertial>
-    <visual>
-      <origin xyz="0 0 0" rpy="0 0 0" />
-      <geometry>
-        <box size="0.01 0.01 0.01" />
-      </geometry>
-      <material name="">
-        <color rgba="0.792156862745098 0.819607843137255 0.933333333333333 1" />
-      </material>
-    </visual>
-    <collision>
-      <origin xyz="0 0 0" rpy="0 0 0" />
-      <geometry>
-        <box size="0.01 0.01 0.01" />
-      </geometry>
-    </collision>
-  </link>
-  <joint name="steering_wheel_joint" type="revolute">
-    <origin xyz="0 0.46 0.15" rpy="1.5708 0 0" />
+  <link name="laser_link">
+    <collision>
+      <origin xyz="0 0 0" rpy="0 0 0" />
+      <geometry>
+        <cylinder length="0.01" radius="0.01" />
+      </geometry>
+    </collision>
+    <visual>
+      <geometry>
+        <cylinder length="0.01" radius="0.01" />
+      </geometry>
+      <material name="Grey" />
+    </visual>
+    <inertial>
+      <origin xyz="0 0 0" rpy="0 0 0" />
+      <mass value="0.1" />
+      <inertia ixx="0.00001" ixy="0.0" ixz="0.0" iyy="0.00001" iyz="0.0" izz="0.00001" />
+    </inertial>
+  </link>
+  <joint name="laser_joint" type="fixed">
+    <origin xyz="0.565 0 0.26" rpy="0 0 0" />
     <parent link="base_link" />
-    <child link="steering_wheel_link" />
-    <axis xyz="0 1 0" />
-    <limit lower="-0.36" upper="0.36" effort="5" velocity="1.0" />
-    <dynamics damping="0.1" friction="1.0" />
-  </joint>
-  <link name="front_wheels_link">
-    <inertial>
-      <origin
-        xyz="0 0 0"
-        rpy="0 0 1.57" />
-      <mass value="0.379124506048444" />
-      <inertia ixx="0.00001697" ixy="0.0" ixz="0.0" iyy="0.01254" iyz="0.0" izz="0.01254" />
-    </inertial>
-    <visual>
-      <origin xyz="0 0 0" rpy="0 1.57 0" />
-      <geometry>
-        <cylinder radius="0.07" length="0.45" />
-      </geometry>
-      <material name="">
-        <color rgba="0.792156862745098 0.819607843137255 0.933333333333333 1" />
-      </material>
-    </visual>
-    <collision>
-      <origin xyz="0 0 0" rpy="0 1.57 0" />
-      <geometry>
-        <cylinder radius="0.07" length="0.45" />
-      </geometry>
-    </collision>
-  </link>
-  <joint name="front_wheels_joint" type="continuous">
-    <origin
-      xyz="0 -0.06 0"
-      rpy="0 0 0" />
-    <parent link="steering_wheel_link" />
-    <child link="front_wheels_link" />
-    <axis xyz="-1 0 0" />
-    <dynamics damping="0.1" friction="1.0" />
-  </joint>
-  <!-- Wheels -->
-  <link name="front_left_wheel_link">
-    <inertial>
-      <origin
-        xyz="-0.175 0 0"
-        rpy="0 0 0" />
-      <mass value="0.379124506048444" />
-      <inertia
-        ixx="0.00135623331658277"
-        ixy="-2.05858146537997E-08"
-        ixz="2.75425144310775E-07"
-        iyy="0.00074553860560749"
-        iyz="-2.05160697747808E-08"
-        izz="0.000744863292198173" />
-    </inertial>
-    <visual>
-      <origin
-        xyz="-0.165 0 0"
-        rpy="0 1.57 0" />
-      <geometry>
-        <cylinder radius="${wheel_radius}" length="${wheel_length}" />
-      </geometry>
-      <material name="">
-        <color rgba="0.792156862745098 0.819607843137255 0.933333333333333 1" />
-      </material>
-    </visual>
-    <collision>
-      <origin
-        xyz="-0.165 0 0"
-        rpy="0 1.57 0" />
-      <geometry>
-        <cylinder radius="${wheel_radius}" length="${wheel_length}" />
-      </geometry>
-    </collision>
-  </link>
-  <joint name="front_left_wheel_joint" type="fixed">
-    <origin
-      xyz="-0.1 0 0"
-      rpy="3.14 0 0" />
-    <parent link="front_wheels_link" />
-    <child link="front_left_wheel_link" />
-    <!-- <axis xyz="1 0 0" /> -->
-    <dynamics damping="0.1" friction="1.0" />
-  </joint>
-  <link name="front_right_wheel_link">
-    <inertial>
-      <origin
-        xyz="0.175 0 0"
-        rpy="0 1.57 0" />
-      <mass value="0.379124506048444" />
-      <inertia
-        ixx="0.00135623331658277"
-        ixy="-2.05858146537997E-08"
-        ixz="2.75425144310775E-07"
-        iyy="0.00074553860560749"
-        iyz="-2.05160697747808E-08"
-        izz="0.000744863292198173" />
-    </inertial>
-    <visual>
-      <origin
-        xyz="0.165 0 0"
-        rpy="0 1.57 0" />
-      <geometry>
-        <cylinder radius="${wheel_radius}" length="${wheel_length}" />
-      </geometry>
-      <material name="">
-        <color rgba="0.792156862745098 0.819607843137255 0.933333333333333 1" />
-      </material>
-    </visual>
-    <collision>
-      <origin
-        xyz="0.165 0 0"
-        rpy="0 1.57 0" />
-      <geometry>
-        <cylinder radius="${wheel_radius}" length="${wheel_length}" />
-      </geometry>
-    </collision>
-  </link>
-  <joint name="front_right_wheel_joint" type="fixed">
-    <origin
-      xyz="0.1 0 0"
-      rpy="1.57 3.1416 3.1416" />
-    <parent link="front_wheels_link" />
-    <child link="front_right_wheel_link" />
-    <!-- <axis xyz="1 0 0" /> -->
-    <dynamics damping="0.1" friction="1.0" />
-  </joint>
-  <link name="rear_left_wheel_link">
-    <inertial>
-      <origin
-        xyz="-0.175 4.72112875317676E-05 9.00201436271342E-06"
-        rpy="0 0 0" />
-      <mass value="0.379124506048444" />
-      <inertia
-        ixx="0.00135623331658277"
-        ixy="-2.05858146537997E-08"
-        ixz="2.75425144310775E-07"
-        iyy="0.00074553860560749"
-        iyz="-2.05160697747808E-08"
-        izz="0.000744863292198173" />
-    </inertial>
-    <visual>
-      <origin
-        xyz="-0.165 0 0"
-        rpy="0 1.57 0" />
-      <geometry>
-        <cylinder radius="${wheel_radius}" length="${wheel_length}" />
-      </geometry>
-      <material name="">
-        <color rgba="0.792156862745098 0.819607843137255 0.933333333333333 1" />
-      </material>
-    </visual>
-    <collision>
-      <origin
-        xyz="-0.165 0 0"
-        rpy="0 1.57 0" />
-      <geometry>
-        <cylinder radius="${wheel_radius}" length="${wheel_length}" />
-      </geometry>
-    </collision>
-  </link>
-  <joint name="rear_left_wheel_joint" type="continuous">
-    <origin
-      xyz="-0.1 0.01 0.09"
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
File: src/segwayrmp_description/urdf/segwayrmp_xacro.xacro (robot description, xacro)
@@ -25,5 +25,5 @@
       <child link="${wheel_prefix}_wheel_link" />
       <xacro:insert_block name="joint_pose" />
-      <axis xyz="${reflect*1} 0 0" />
+      <axis xyz="0 ${reflect*1} 0" />
     </joint>
   </xacro:macro>
@@ -52,5 +52,5 @@
       <child link="${steering_prefix}_link" />
       <xacro:insert_block name="joint_pose" />
-      <axis xyz="0 1 0" />
+      <axis xyz="0 0 1" />
       <limit lower="-0.36" upper="0.36" effort="0" velocity="1.0" />
     </joint>

Commit message: nav2_params.yaml: tuned controller and planner

File: src/segwayrmp_description/urdf/segwayrmp.urdf.xacro (robot description, xacro)
@@ -106,10 +106,10 @@
     </inertial>
   </link>
-  <joint name="steering_joint" type="revolute">
+  <joint name="steering_joint" type="continuous">
     <origin xyz="0.25 0 -0.09" rpy="0 0 0" />
     <parent link="base_footprint" />
     <child link="steering_link" />
     <axis xyz="0 0 1" />
-    <limit lower="-0.36" upper="0.36" effort="0.0" velocity="0.0" />
+    <!-- <limit lower="-0.36" upper="0.36" effort="0.0" velocity="0.0" /> -->
     <dynamics damping="0.2" />
   </joint>
